File: painemittari.kicad_sch (KiCad schematic)
At the start: 18 parts, among them U1 TL431, U2 MCP1700-3302E/TO, U3 MCP6002-I/P, U4 SDP816-125Pa

Commit message: Dippadappa
Connections:
- net VCC 3V3 is gone; now on net +3V3: C2.1, U2.3 (VO)
- net VCC renamed +3V3
Other:
- note added: "Adjust to ~11.5 % so that Out+ = Out- when dP = 0. For easier (less sensitive) trimming, use 100 k resistor to VCC and 20 k trimmer to GND. 100 k + 13 k fixed resistors could also work, but good luck getting zero offset at output!"
- note added: "LED lits when battery voltage exceeds ~4 V"
- note removed: "Adjust to ~11.5 % so that Out+ = Out- when dP = 0. For easier (less sensitive) trimming, use 100 k resistor to VCC and 20 k trimmer to GND. 100 k + 13 k fixed resistors could also work, but getting getting exact match at output requires good luck!"
- note removed: "LED lits when battery voltage exceeds 3.68 V"
- moved on the sheet: R2

Commit message: Update painemittari.kicad_sch
Other:
- note added: "~381 mV"
- note removed: "~380 mV"
Changed lines of the file:
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@@
 		)
 	)
-	(text "~380 mV"
+	(text "~381 mV"
 		(exclude_from_sim no)
 		(at 136.906 88.138 0)

Commit message: Blah
Parts:
- U1: value TL431 -> TL431CZ
Other:
- note added: "Adjust RV1 to ~11.5 % so that Out+ = Out- when dP = 0. For easier (less sensitive) trimming, use 100 k resistor to VCC and 20 k trimmer to GND."
- note added: "C3 is optional."
- note added: "LED lits when battery voltage is sufficient."
- note removed: "Adjust to ~11.5 % so that Out+ = Out- when dP = 0. For easier (less sensitive) trimming, use 100 k resistor to VCC and 20 k trimmer to GND. 100 k + 13 k fixed resistors could also work, but good luck getting zero offset at output!"
- note removed: "C3 is optional. 1 µF filters out noise above ~3 Hz."
- note removed: "LED lits when battery voltage exceeds ~4 V"
- note removed: "Using 110 k + 150 k, both in E24, scaling is within 0.2 % from ideal 0.5757...."
- title: Differential Pressure Probe / Micromanometer -> Differential Pressure Probe
- moved on the sheet: C1, C2, C3, R4, R5, R6, R7, RV1, U3A, U3B, U3C, U4
